File: Schematic/motor.kicad_pcb (KiCad board)
At the start: 2 copper layers, 45 x 45 mm, 48 parts, among them J1 CONN_02X05, J11 V, J12 U, J13 W, J2 RS485, J3 RS485, J6 12, J9 GND, Q1 PSMN3R3-40YS, Q2 PSMN3R3-40YS, Q3 PSMN3R3-40YS, Q4 PSMN3R3-40YS, Q5 PSMN3R3-40YS, Q6 PSMN3R3-40YS, U1 STSPIN32F0, U2 LTC2876, U3 MA700, Y1 8Mhz

Commit message: Start of work to use the stspin32g4
Other:
- net class Default removed
